File: T3-Redstone/kicad/t3-redstone.kicad_sch (KiCad schematic)
At the start: 87 parts, among them J1 Gemstone 40P disi, J10 QWIIC, J11 USB-C, J12 ACIL STOP (NC), J13 BUMPER, J14 GPIO, J2 XT60 2S LiPo, J3 GEMSTONE GUC, J4 MOTOR A, J5 MOTOR B, J6 ENKODER A, J7 ENKODER B, J8A SERVO 1-8, J8B SERVO 9-16, Q1 AO4407A, Q2 AO4407A, Q3 AO3400A, Q4 AO3400A, SW1 BOOT, SW2 RESET, U1 ESP32-S3-WROOM-1U-N8R2, U10 USBLC6-2SC6, U2 DRV8874, U3 DRV8874, U4 PCA9685PW, U5 INA226, U6 AP2112K-3.3, U7 TPS563201, U8 74LVC245, U9 74AHCT1G125

Commit message: T3-Redstone: guc dagitimi ve yonlendirme duzeltmeleri (ara kayit)
- +3V3 omurgasi B.Cu'ya tasindi; LDO cikisi, I2C pull-up, PCA9685, INA226 adres
  pinleri ve sag bolge icin kilitli baglantilar
- C2 / C4 ters yonluydu (3V3 pini GND tarafinda), C12 cipten 11 mm uzaktaydi
- LED +5V pinleri kesitin ustundeki F.Cu raydan birlesiyor
- USB D+/D- icin ayri net sinifi (0.1 mm aralik)
- rs_route: fanout pedin kendisini engel sayiyordu (SWIG 'is' karsilastirmasi);
  pasiflerin guc pinleri yonlendirmeden once fanout'lanir; ayni netin kopuk
  parcalarini birlestiren onarim adimi

Co-Authored-By: Claude Opus 5.5 <noreply@anthropic.com>
Claude-Session: https://claude.ai/code/session_01YQNy21SHVjiYix4RbadZre
Parts:
- removed RS1: 2m 2W, Resistor_SMD:R_2512_6332Metric, symbol Device:R
- added RS1: 2m 3W, Resistor_SMD:R_Shunt_Vishay_WSK2512_6332Metric_T1.19mm, symbol Device:R_Shunt
Connections:
- net BUMP1: now also U1.7 (IO7); no longer U1.31 (IO38)
- net BUMP2: now also U1.8 (IO15); no longer U1.32 (IO39)
- net DRV_nFAULT: now also U1.22 (IO14); no longer U1.9 (IO16)
- net DRV_nSLEEP: now also U1.21 (IO13); no longer U1.8 (IO15)
- net ENC_A1: now also U1.31 (IO38); no longer U1.12 (IO8)
- net ENC_A2: now also U1.33 (IO40); no longer U1.18 (IO10)
- net ENC_B1: now also U1.32 (IO39); no longer U1.17 (IO9)
- net ENC_B2: now also U1.34 (IO41); no longer U1.19 (IO11)
- net ESTOP_LOOP: now also U1.6 (IO6); no longer U1.11 (IO18)
- net ESTOP_STAT: now also U1.37 (TXD0); no longer U1.20 (IO12)
- net HOST_RX: now also U1.4 (IO4); no longer U1.24 (IO47)
- net HOST_TX: now also U1.5 (IO5); no longer U1.25 (IO48)
- net I2C_SCL: now also U1.36 (RXD0); no longer U1.35 (IO42)
- net I2C_SDA: now also U1.35 (IO42); no longer U1.34 (IO41)
- net LED_DATA: now also U1.24 (IO47); no longer U1.33 (IO40)
- net MA_EN: now also U1.18 (IO10); no longer U1.5 (IO5)
- net MA_PH: now also U1.17 (IO9); no longer U1.4 (IO4)
- net MB_EN: now also U1.20 (IO12); no longer U1.7 (IO7)
- net MB_PH: now also U1.19 (IO11); no longer U1.6 (IO6)
- net PWR_ALERT: now also U1.25 (IO48); no longer U1.22 (IO14)
- net VBAT: now also RS1.1; no longer U5.10 (Vin+)
- net VSYS: now also RS1.4; no longer U5.8 (Vbus), U5.9 (Vin-)
- net GPIO13 renamed GPIO16
- net GPIO16: now also U1.9 (IO16); no longer U1.21 (IO13)
- new net SNS_N: RS1.3, U5.8 (Vbus), U5.9 (Vin-)
- new net SNS_P: RS1.2, U5.10 (Vin+)
